File: pcb/front_panel.kicad_sch (KiCad schematic)
At the start: 11 parts, among them J3 DB9_Female, J4 DB9_Male, J5 Conn_2Rows-09Pins, M1 Stepper_Motor_bipolar, SW2 SW_DPDT_x2, U1 L293D

Commit message: Finishing PCB traces
Parts:
- added J6: Conn_01x04, Connector_PinHeader_2.54mm:PinHeader_1x04_P2.54mm_Vertical, symbol Connector_Generic:Conn_01x04
- added J7: Conn_01x04, Connector_PinHeader_2.54mm:PinHeader_1x04_P2.54mm_Horizontal, symbol Connector_Generic:Conn_01x04
- D101: symbol Device:D_Bridge_+AA- -> Device:D_Bridge_+-AA
- M1: footprint Connector_PinHeader_2.54mm:PinHeader_1x04_P2.54mm_Vertical -> local:auto_stepper_backing
Connections:
- net +5V: no longer J4.3, J5.9 (Pin_9)
- net at D101.2 (-): now also D102.1 (K); no longer J3.4
- net at D101.3: now also J3.4; no longer J3.8
- net at D101.4: now also J3.8; no longer D102.1 (K)
- net at U1.11 (3Y): now also J6.3 (Pin_3); no longer M1.3
- net at U1.14 (4Y): now also J6.4 (Pin_4); no longer M1.4
- net at U1.3 (1Y): now also J6.1 (Pin_1); no longer M1.1
- net at U1.6 (2Y): now also J6.2 (Pin_2); no longer M1.2 (-)
- new net: J7.1 (Pin_1), M1.1
- new net: J7.2 (Pin_2), M1.2 (-)
- new net: J7.3 (Pin_3), M1.3
- new net: J7.4 (Pin_4), M1.4
- new net +5V_NC: J4.3, J5.9 (Pin_9)
Other:
- moved on the sheet: M1, RV1, RV2
